Commit message: rebel_description: restructure description

File: rebel_description/urdf/igus_rebel.control.xacro (robot description, xacro)
@@ -2,26 +2,110 @@
 <!-- igus_rebel.control.xacro -->
 <robot xmlns:xacro="http://www.ros.org/wiki/xacro">
-    <xacro:macro name="igus_rebel_control" params="arm_id">
-        <xacro:macro name="arm_control" params="transmission joint motor">
-            <transmission name="${transmission}">
-                <type>transmission_interface/SimpleTransmission</type>
-                <joint name="${joint}">
-                    <hardwareInterface>hardware_interface/EffortJointInterface</hardwareInterface>
-                </joint>
-                <actuator name="${motor}">
-                    <hardwareInterface>hardware_interface/EffortJointInterface</hardwareInterface>
-                    <mechanicalReduction>1</mechanicalReduction>
-                </actuator>
-            </transmission>
-        </xacro:macro>
-        <xacro:arm_control transmission="${arm_id}_tran_1" joint="joint1" motor="${arm_id}_motor_1"/>
-        <xacro:arm_control transmission="${arm_id}_tran_2" joint="joint2" motor="${arm_id}_motor_2"/>
-        <xacro:arm_control transmission="${arm_id}_tran_3" joint="joint3" motor="${arm_id}_motor_3"/>
-        <xacro:arm_control transmission="${arm_id}_tran_4" joint="joint4" motor="${arm_id}_motor_4"/>
-        <xacro:arm_control transmission="${arm_id}_tran_5" joint="joint5" motor="${arm_id}_motor_5"/>
-        <xacro:arm_control transmission="${arm_id}_tran_6" joint="joint6" motor="${arm_id}_motor_6"/>
-        <gazebo>
-            <plugin name="gazebo_ros_control" filename="libgazebo_ros_control.so"/>
-        </gazebo>
-    </xacro:macro>
+<xacro:macro name="igus_rebel_control">
+     <xacro:property name="name" value="igus_rebel" />
+     <xacro:property name="ns" value="" />
+     <xacro:property name="ip_address" value="192.168.3.11" />
+     <xacro:property name="use_fake_hardware" value="true" />
+     <xacro:property name="mock_sensor_commands" value="false" />
+    <ros2_control name="${name}" type="system">
+      <hardware>
+        <plugin>ros2_control_demo_example_7/RobotSystem</plugin>
+      </hardware>
+      <xacro:macro name="configure_joint" params="joint_name initial_position">
+        <joint name="${joint_name}">
+          <param name="initial_position">${initial_position}</param>
+          <command_interface name="position"/>
+          <command_interface name="velocity"/>
+          <command_interface name="effort"/>
+          <state_interface name="position"/>
+          <state_interface name="velocity"/>
+          <state_interface name="effort"/>
+        </joint>
+      </xacro:macro>
+      <joint name="joint_1">
+        <command_interface name="position">
+          <param name="min">{-2*pi}</param>
+          <param name="max">{2*pi}</param>
+        </command_interface>
+        <command_interface name="velocity">
+          <param name="min">-3.15</param>
+          <param name="max">3.15</param>
+        </command_interface>
+        <state_interface name="position">
+          <param name="initial_value">0.0</param>
+        </state_interface>
+        <state_interface name="velocity"/>
+      </joint>
+      <joint name="joint_2">
+        <command_interface name="position">
+          <param name="min">{-2*pi}</param>
+          <param name="max">{2*pi}</param>
+        </command_interface>
+        <command_interface name="velocity">
+          <param name="min">-3.15</param>
+          <param name="max">3.15</param>
+        </command_interface>
+        <state_interface name="position">
+          <param name="initial_value">0.0</param>
+        </state_interface>
+        <state_interface name="velocity"/>
+      </joint>
+      <joint name="joint_3">
+        <command_interface name="position">
+          <param name="min">{-pi}</param>
+          <param name="max">{pi}</param>
+        </command_interface>
+        <command_interface name="velocity">
+          <param name="min">-3.15</param>
+          <param name="max">3.15</param>
+        </command_interface>
+        <state_interface name="position">
+          <param name="initial_value">0.0</param>
+        </state_interface>
+        <state_interface name="velocity"/>
+      </joint>
+      <joint name="joint_4">
+        <command_interface name="position">
+          <param name="min">{-2*pi}</param>
+          <param name="max">{2*pi}</param>
+        </command_interface>
+        <command_interface name="velocity">
+          <param name="min">-3.2</param>
+          <param name="max">3.2</param>
+        </command_interface>
+        <state_interface name="position">
+          <param name="initial_value">0.0</param>
+        </state_interface>
+        <state_interface name="velocity"/>
+      </joint>
+      <joint name="joint_5">
+        <command_interface name="position">
+          <param name="min">{-2*pi}</param>
+          <param name="max">{2*pi}</param>
+        </command_interface>
+        <command_interface name="velocity">
+          <param name="min">-3.2</param>
+          <param name="max">3.2</param>
+        </command_interface>
+        <state_interface name="position">
+          <param name="initial_value">0.0</param>
+        </state_interface>
+        <state_interface name="velocity"/>
+      </joint>
+      <joint name="joint_6">
+        <command_interface name="position">
+          <param name="min">{-2*pi}</param>
+          <param name="max">{2*pi}</param>
+        </command_interface>
+        <command_interface name="velocity">
+          <param name="min">-3.2</param>
+          <param name="max">3.2</param>
+        </command_interface>
+        <state_interface name="position">
+          <param name="initial_value">0.0</param>
+        </state_interface>
+        <state_interface name="velocity"/>
+      </joint>
+    </ros2_control>
+  </xacro:macro>
 </robot>

File: rebel_description/urdf/igus_rebel.urdf (robot description, URDF)
Before this commit: robot igus_rebel, 9 links, 8 joints
Links:
- removed link rebel_link1
- removed link rebel_link2
- removed link rebel_link3
- removed link rebel_link4
- removed link rebel_link5
- removed link rebel_link6
- removed link rebel_link7
- removed link rebel_link8
- added link ft_frame
- added link link_1, mass 0.1; collision mesh filename=package://rebel_description/meshes/robolink_rebel/Robolink_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; visual mesh filename=package://rebel_description/meshes/robolink_rebel/Robolink_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
- added link link_2, mass 0.1; collision mesh filename=package://rebel_description/meshes/robolink_rebel/Robolink_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; visual mesh filename=package://rebel_description/meshes/robolink_rebel/Robolink_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
- added link link_3, mass 0.1; collision mesh filename=package://rebel_description/meshes/robolink_rebel/Robolink_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; visual mesh filename=package://rebel_description/meshes/robolink_rebel/Robolink_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
- added link link_4, mass 0.1; collision mesh filename=package://rebel_description/meshes/robolink_rebel/Robolink_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; visual mesh filename=package://rebel_description/meshes/robolink_rebel/Robolink_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
- added link link_5, mass 0.1; collision mesh filename=package://rebel_description/meshes/robolink_rebel/Robolink_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; visual mesh filename=package://rebel_description/meshes/robolink_rebel/Robolink_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
- added link link_6, mass 0.1; collision mesh filename=package://rebel_description/meshes/robolink_rebel/Robolink_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; visual mesh filename=package://rebel_description/meshes/robolink_rebel/Robolink_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
- added link link_7, mass 0.1; collision mesh filename=package://rebel_description/meshes/robolink_rebel/Robolink_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; visual mesh filename=package://rebel_description/meshes/robolink_rebel/Robolink_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
- added link link_8, mass 0.1; collision mesh filename=package://rebel_description/meshes/robolink_rebel/Robolink_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; visual mesh filename=package://rebel_description/meshes/robolink_rebel/Robolink_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
- added link tool0
Joints:
- removed joint joint1
- removed joint joint2
- removed joint joint3
- removed joint joint4
- removed joint joint5
- removed joint joint6
- added joint base_joint: type fixed, parent world, child base_link, origin xyz=0 0 0 rpy=0 0 0, axis 0 0 1
- added joint joint-ft_frame: type fixed, parent link_6, child ft_frame, origin xyz=0 0 0 rpy=0 0 0
- added joint joint-tool: type fixed, parent ft_frame, child tool0, origin xyz=0 0 .185 rpy=0 0 0
- added joint joint_1: type revolute, parent base_link, child link_1, origin xyz=0.0 0 0.126 rpy=0.0 0.0 3.1416, axis 0 0 -1, limit lower=${-pi} upper=${pi} effort=1000.0 velocity=2.5
- added joint joint_2: type revolute, parent link_1, child link_2, origin xyz=0.0 0.025 0.153 rpy=0.0 0.0 0.0, axis 0 -1 0, limit lower=${-pi} upper=${pi} effort=1000.0 velocity=2.5
- added joint joint_3: type revolute, parent link_4, child link_5, origin xyz=0.0 0.025 0.1 rpy=0.0 0.0 0.0, axis 0 -1 0, limit lower=${-pi} upper=${pi} effort=1000.0 velocity=2.5
- added joint joint_4: type revolute, parent link_5, child link_6, origin xyz=0.0 -0.025 0.153 rpy=0.0 0.0 0.0, axis 0 0 1, limit lower=${-pi} upper=${pi} effort=1000.0 velocity=2.5
- added joint joint_5: type revolute, parent link_6, child link_7, origin xyz=0.0 0.029 0.143 rpy=0.0 0.0 0.0, axis 0 -1 0, limit lower=${-pi} upper=${pi} effort=1000.0 velocity=2.5
- added joint joint_6: type revolute, parent link_7, child link_8, origin xyz=0.0 -0.029 0.1188 rpy=0.0 0.0 0.0, axis 0 0 1, limit lower=${-pi} upper=${pi} effort=1000.0 velocity=2.5
- joint joint_fixed_1: child rebel_link3 -> link_3; parent rebel_link2 -> link_2
- joint joint_fixed_2: child rebel_link4 -> link_4; parent rebel_link3 -> link_3

File: rebel_description/urdf/igus_rebel_robot.urdf.xacro (robot description, xacro)
@@ -5,5 +5,5 @@
   <xacro:include filename="$(find rebel_description)/urdf/igus_rebel.urdf" />
   <xacro:include filename="$(find rebel_description)/urdf/igus_rebel.control.xacro"/>
-  <xacro:igus_rebel_control arm_id="igus_rebel"/>
+  <xacro:igus_rebel_control />
   <link name="world" />
   <joint name="world_joint" type="fixed">

Commit message: dirty fixup

File: rebel_description/urdf/igus_rebel.control.xacro (robot description, xacro)
@@ -8,8 +8,10 @@
      <xacro:property name="use_fake_hardware" value="true" />
      <xacro:property name="mock_sensor_commands" value="false" />
+     <xacro:property name="port" value="3920" />
     <ros2_control name="${name}" type="system">
       <hardware>
         <xacro:if value="${use_fake_hardware}">
-          <plugin>fake_components/GenericSystem</plugin>
+        <plugin>mock_components/GenericSystem</plugin>
+        <param name="mimic">joint1</param>
           <param name="mock_sensor_commands">${mock_sensor_commands}</param>
           <param name="state_following_offset">0.0</param>

File: rebel_description/urdf/igus_rebel.urdf (robot description, URDF)
Before this commit: robot igus_rebel, 11 links, 11 joints
Links:
- added link world

File: rebel_description/urdf/igus_rebel_robot.urdf.xacro (robot description, xacro)
@@ -4,11 +4,3 @@
   <!-- igus_rebel -->
   <xacro:include filename="$(find rebel_description)/urdf/igus_rebel.urdf" />
-  <xacro:include filename="$(find rebel_description)/urdf/igus_rebel.control.xacro"/>
-  <xacro:igus_rebel_control />
-  <link name="world" />
-  <joint name="world_joint" type="fixed">
-    <parent link="world" />
-    <child link = "base_link" />
-    <origin xyz="0.0 0.0 0.0" rpy="0.0 0.0 0.0" />
-  </joint>
 </robot>
